File: TeensyPrototypeBoard.brd (EAGLE design)
At the start: 58.3 x 51.7 mm, 50 parts, among them Q1 16mhz, SW1 SPST_TACT-KMR2, SW2 SPST_TACT-KMR2, U3 BLE112-A, U4 MPU-6050-1, X1 32.768khz

Commit message: connect the oscillator and add generate BOM.txt
Parts:
- renumbered PROG to PROGRAM_HEADER, U$2 to MINI54_MICRO, U$3 to MICRO_SD_CARD_SINK, U4 to IMU
Routing:
- net N$1: track 0.00 -> 4.70 mm
- net N$8: track 0.00 -> 2.87 mm
