File: Eagle_File/TeensyPrototypeBoard.sch (EAGLE design)
At the start: 50 parts, among them Q1 16mhz, SW1 SPST_TACT-KMR2, SW2 SPST_TACT-KMR2, U3 BLE112-A, X1 32.768khz

Commit message: modify the name and value on the board
Parts:
- renumbered JP2 to POWER, U1 to USB
